File: tank.kicad_sch (KiCad schematic)
At the start: 0 parts

Commit message: Ajout du BMS
Parts:
- added J1: USB4230-03-A_REVA, local:GCT_USB4230-03-A_REVA, symbol local:USB4230-03-A_REVA
Connections:
- new net GND: J1.A1 (GND_A), J1.A12 (GND_A), J1.B1 (GND_B), J1.B12 (GND_B), J1.SH1 (SHIELD), J1.SH2 (SHIELD), J1.SH3 (SHIELD), J1.SH4 (SHIELD)
- new net USB_CC1: J1.A5 (CC1)
- new net USB_CC2: J1.B5 (CC2)
- new net USB_D+: J1.A6 (DP1), J1.B6 (DP2)
- new net USB_D-: J1.A7 (DN1), J1.B7 (DN2)
- new net VBUS_A: J1.A4 (VBUS_A), J1.A9 (VBUS_A), J1.B4 (VBUS_B), J1.B9 (VBUS_B)
- no-connect marks 0 -> 10
Other:
- sheet power ports: added USB_CC1, USB_CC2, VBUS_USB; removed none
