File: bms.kicad_sch (KiCad schematic)
At the start: 77 parts, among them IC4 BQ24810RUYR, J4 S4B-XH-A-1, SW1 B3S-1000, U1 XSM6K519NW, U2 XSM6K519NW, U3 XSM6K519NW, U4 XSM6K519NW, U5 XSM6K519NW, U6 BQ76905RGRR, U7 XSM6K519NW, U8 XSM6K519NW

Commit message: Minor Schematics update
Parts:
- removed D9: LM4040DIM3-2.5/NOPB, local:SOT95P237X112-3N, symbol Device:D_Zener
- added D4: LM4040, local:SOT95P237X112-3N, symbol local:LM4040
- C14: renamed from C12; footprint Capacitor_SMD:C_0805_2012Metric -> Capacitor_SMD:C_0603_1608Metric; symbol local:C_0402 -> local:C
- C15: renamed from C13; footprint Capacitor_SMD:C_0805_2012Metric -> Capacitor_SMD:C_0603_1608Metric; symbol local:C_0402 -> local:C
- C16: renamed from C14; footprint Capacitor_SMD:C_0805_2012Metric -> Capacitor_SMD:C_0603_1608Metric; symbol local:C_0402 -> local:C
- C17: renamed from C52; symbol local:C_0402 -> local:C
- C18: renamed from C53; symbol local:C_0402 -> local:C
- C19: renamed from C15; footprint Capacitor_SMD:C_0805_2012Metric -> Capacitor_SMD:C_0603_1608Metric; symbol local:C_0402 -> local:C
- C20: renamed from C16; footprint Capacitor_SMD:C_0805_2012Metric -> Capacitor_SMD:C_0603_1608Metric; symbol local:C_0402 -> local:C
- C21: renamed from C17; footprint Capacitor_SMD:C_0805_2012Metric -> Capacitor_SMD:C_0603_1608Metric; symbol local:C_0402 -> local:C
- C22: renamed from C18; footprint Capacitor_SMD:C_0805_2012Metric -> Capacitor_SMD:C_0603_1608Metric; symbol local:C_0402 -> local:C
- C23: renamed from C20; footprint Capacitor_SMD:C_0805_2012Metric -> Capacitor_SMD:C_0603_1608Metric; symbol local:C_0402 -> local:C
- C24: renamed from C19; footprint Capacitor_SMD:C_0805_2012Metric -> Capacitor_SMD:C_0603_1608Metric; symbol local:C_0402 -> local:C
- C25: renamed from C21; footprint Capacitor_SMD:C_0805_2012Metric -> Capacitor_SMD:C_0603_1608Metric; symbol local:C_0402 -> local:C
- C26: renamed from C22; footprint Capacitor_SMD:C_0805_2012Metric -> Capacitor_SMD:C_0603_1608Metric; symbol local:C_0402 -> local:C
- C27: renamed from C23; symbol local:C_0402 -> local:C
- C28: renamed from C50; symbol local:C_0402 -> local:C
- C29: renamed from C24; footprint Capacitor_SMD:C_0805_2012Metric -> Capacitor_SMD:C_0603_1608Metric; symbol local:C_0402 -> local:C
- C30: renamed from C27; footprint Capacitor_SMD:C_0805_2012Metric -> Capacitor_SMD:C_0603_1608Metric; symbol local:C_0402 -> local:C
- C31: renamed from C28; footprint Capacitor_SMD:C_0805_2012Metric -> Capacitor_SMD:C_0603_1608Metric; symbol local:C_0402 -> local:C
- C32: renamed from C54; footprint Capacitor_SMD:C_0805_2012Metric -> Capacitor_SMD:C_0603_1608Metric; symbol local:C_0402 -> local:C
- C33: renamed from C29; footprint Capacitor_SMD:C_0805_2012Metric -> Capacitor_SMD:C_0603_1608Metric; symbol local:C_0402 -> local:C
- C34: renamed from C30; footprint Capacitor_SMD:C_0805_2012Metric -> Capacitor_SMD:C_0603_1608Metric; symbol local:C_0402 -> local:C
- C35: renamed from C31; footprint Capacitor_SMD:C_0805_2012Metric -> Capacitor_SMD:C_0603_1608Metric; symbol local:C_0402 -> local:C
- C36: renamed from C32; footprint Capacitor_SMD:C_0805_2012Metric -> Capacitor_SMD:C_0603_1608Metric; symbol local:C_0402 -> local:C
- C37: renamed from C33; footprint Capacitor_SMD:C_0805_2012Metric -> Capacitor_SMD:C_0603_1608Metric; symbol local:C_0402 -> local:C
- C38: renamed from C34; footprint Capacitor_SMD:C_0805_2012Metric -> Capacitor_SMD:C_0603_1608Metric; symbol local:C_0402 -> local:C
- C39: renamed from C35; footprint Capacitor_SMD:C_0805_2012Metric -> Capacitor_SMD:C_0603_1608Metric; symbol local:C_0402 -> local:C
- C40: renamed from C36; footprint Capacitor_SMD:C_0805_2012Metric -> Capacitor_SMD:C_0603_1608Metric; symbol local:C_0402 -> local:C
- IC4: value BQ24810RUYR -> BQ24800RUYR
- J6: renamed from J4; footprint S4B-XH-A-1:JST_S4B-XH-A-1 -> local:JST_S4B-XH-A-1
- R17: renamed from R9; footprint Resistor_SMD:R_0805_2012Metric -> local:RESC6331X88N
- R18: renamed from R10; footprint Resistor_SMD:R_0805_2012Metric -> Resistor_SMD:R_0603_1608Metric
- R19: renamed from R11; footprint Resistor_SMD:R_0805_2012Metric -> Resistor_SMD:R_0603_1608Metric
- R20: renamed from R12; footprint Resistor_SMD:R_0805_2012Metric -> Resistor_SMD:R_0603_1608Metric
- R21: renamed from R13; footprint Resistor_SMD:R_0805_2012Metric -> Resistor_SMD:R_0603_1608Metric
- R22: renamed from R14; footprint Resistor_SMD:R_0805_2012Metric -> Resistor_SMD:R_0603_1608Metric
- R23: renamed from R15; footprint Resistor_SMD:R_0805_2012Metric -> Resistor_SMD:R_0603_1608Metric
- R24: renamed from R16; footprint Resistor_SMD:R_0805_2012Metric -> Resistor_SMD:R_0603_1608Metric
- R25: renamed from R17; footprint Resistor_SMD:R_0805_2012Metric -> Resistor_SMD:R_0603_1608Metric
- R26: renamed from R18; footprint Resistor_SMD:R_0805_2012Metric -> local:RESC6331X88N
- R27: renamed from R19; footprint Resistor_SMD:R_0805_2012Metric -> Resistor_SMD:R_0603_1608Metric
- R28: renamed from R20; footprint Resistor_SMD:R_0805_2012Metric -> Resistor_SMD:R_0603_1608Metric
- R29: renamed from R21; footprint Resistor_SMD:R_0805_2012Metric -> Resistor_SMD:R_0603_1608Metric
- R30: renamed from R22; footprint Resistor_SMD:R_0805_2012Metric -> Resistor_SMD:R_0603_1608Metric
- R31: renamed from R24; footprint Resistor_SMD:R_0805_2012Metric -> Resistor_SMD:R_0603_1608Metric
- R32: renamed from R25; footprint Resistor_SMD:R_0805_2012Metric -> Resistor_SMD:R_0603_1608Metric
- R34: renamed from R27; footprint Resistor_SMD:R_0805_2012Metric -> Resistor_SMD:R_0603_1608Metric
- R36: renamed from R29; footprint Resistor_SMD:R_0805_2012Metric -> Resistor_SMD:R_0603_1608Metric
- R37: renamed from R30; footprint Resistor_SMD:R_0805_2012Metric -> Resistor_SMD:R_0603_1608Metric
- R39: renamed from R44; footprint Resistor_SMD:R_0805_2012Metric -> Resistor_SMD:R_0603_1608Metric
- R40: renamed from R32; footprint Resistor_SMD:R_0805_2012Metric -> Resistor_SMD:R_0603_1608Metric
- R41: renamed from R33; footprint Resistor_SMD:R_0805_2012Metric -> Resistor_SMD:R_0603_1608Metric
- R42: renamed from R45; footprint Resistor_SMD:R_0805_2012Metric -> Resistor_SMD:R_0603_1608Metric
- R43: renamed from R34; footprint Resistor_SMD:R_0805_2012Metric -> Resistor_SMD:R_0603_1608Metric
- R44: renamed from R35; footprint Resistor_SMD:R_0805_2012Metric -> Resistor_SMD:R_0603_1608Metric
- R45: renamed from R36; value 0.001 -> 0.01; footprint Resistor_SMD:R_0805_2012Metric -> local:RESC6331X88N
- TP1, TP2, TP5, TP6: footprint (none) -> TestPoint:TestPoint_Pad_D1.0mm
- TP3, TP4: footprint (none) -> TestPoint:TestPoint_THTPad_D4.0mm_Drill2.0mm
- renumbered R26 to R33, R28 to R35, R31 to R38
Connections:
- net +BATT is gone; now on net V_BATT: C38.2, TP3.1, U6.17 (BAT)
- net -BATT: now also U7.8; no longer U7.7
- net GND: now also U5.8, D4.2 (A), D4.3 (*); no longer U5.7
- net ILIM: now also D4.1 (K)
- net V_BATT: no longer C27.2, C28.2
- net V_BMS_IN: now also U1.7; no longer U1.8
- net V_BMS_OUT: now also U3.7, U4.7; no longer U3.8, U4.8
- net at C24.1, IC4.27 (PHASE), L3.1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: now also U4.8, U5.7; no longer U4.7, U5.8
- net V_SYS_SN: now reaches C20.2, C22.2, IC4.1 (ACN), R19.2
- net V_SYS_SP: now reaches C20.1, C21.2, IC4.2 (ACP), R18.2
- net at C23.1, C25.2, L3.2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: now also C27.2, C28.2, U3.8; no longer U3.7
- net at C16.1, R22.1, U1.4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: now also U1.8, U2.8; no longer U1.7, U2.7
- net V_BATT_SP: now reaches C36.2, C37.2, R43.1, U6.10 (CHG)
- net V_BATT_SP: now also C25.1, R27.2
- net at R43.2, R45.1, U8.4: now also U8.8; no longer U8.7
- net at R17.2, R18.1, U2.1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: now also U2.7; no longer U2.8
- net at U7.1, U7.2, U7.5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: now also U7.7, U8.7; no longer U7.8, U8.8
- net V_BATT_SN: now reaches C36.1, C37.1, R44.1, U6.9 (DSG)
- net V_BATT_SN: now also C26.1, R28.2
Other:
- moved on the sheet: C23, C25, C26, C27, C28, R26, U3

Commit message: Modification mineur du schéma, ajout du PCB V1
Parts:
- D2, D3: value ~ -> (none)
Connections:
- net V_BATT_SN: no longer C36.1, C37.1, R44.1, U6.9 (DSG)
- net V_BATT_SP: no longer C36.2, C37.2, R43.1, U6.10 (CHG)
- new net VM_BATT_SN: C36.1, C37.1, R44.1, U6.9 (DSG)
- new net VM_BATT_SP: C36.2, C37.2, R43.1, U6.10 (CHG)
